File: hardware/picoprobe.kicad_sch (KiCad schematic)
At the start: 34 parts, among them J1 Conn_01x04_Pin, J2 Conn_01x03_Pin, J3 Conn_01x03_Pin, J4 Conn_01x03_Pin, U2 74AUP1G17, U3 74AUP1G17

Commit message: Add panelization script and gerber production files
- Add make_smt_sample.py: 2x2 kikit panelization with frame, mousebites,
  tooling holes, and fiducials (panel < 10cm per side)
- Add production gerber ZIP, BOM, positions, and netlist
- Add panelized KiCad PCB files (picoprobe_panel)
- Update .gitignore to exclude KiCad backups and fabrication toolkit
  nested output

Co-Authored-By: Claude Sonnet 4.6 <noreply@anthropic.com>
Parts:
- C1, C2: LCSC Part (none) -> C23733
- C3, C4: LCSC Part (none) -> C307331
- D1: LCSC Part (none) -> C2286
- D2, D4: LCSC Part (none) -> C7496818
- D3, D5: LCSC Part (none) -> C965800
- R1, R10, R2, R9: LCSC Part (none) -> C17168
- R11, R12, R5, R6, R7, R8: LCSC Part (none) -> C25076
- R13, R14, R15, R16, R3: LCSC Part (none) -> C25117
- R17, R18, R19: LCSC Part (none) -> C25900
- U2, U3: footprint Package_TO_SOT_SMD:SOT-23-5 -> Package_TO_SOT_SMD:SOT-353_SC-70-5; LCSC Part (none) -> C48946883

Commit message: Update PCB layout: R18/R19 footprints to 0603, adjust component positions
Co-Authored-By: Claude Sonnet 4.6 <noreply@anthropic.com>
Parts:
- R1, R2: footprint Resistor_SMD:R_0402_1005Metric -> Resistor_SMD:R_0603_1608Metric
Changed lines of the file:
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@@
 			)
 		)
-		(property "Footprint" "Resistor_SMD:R_0402_1005Metric"
+		(property "Footprint" "Resistor_SMD:R_0603_1608Metric"
 			(at 48.26 172.72 0)
 			(hide yes)
@@
 			)
 		)
-		(property "Footprint" "Resistor_SMD:R_0402_1005Metric"
+		(property "Footprint" "Resistor_SMD:R_0603_1608Metric"
 			(at 41.91 172.72 0)
 			(hide yes)

Commit message: Update R18/R19 LCSC part number C17168 to C21189
Co-Authored-By: Claude Sonnet 4.6 <noreply@anthropic.com>
Parts:
- R1, R2: LCSC Part C17168 -> C21189
Changed lines of the file:
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@@
 			)
 		)
-		(property "LCSC Part" "C17168"
+		(property "LCSC Part" "C21189"
 			(at 48.26 172.72 90)
 			(hide yes)
@@
 			)
 		)
-		(property "LCSC Part" "C17168"
+		(property "LCSC Part" "C21189"
 			(at 41.91 172.72 90)
 			(hide yes)
